File: RIO_V1/RIO_V1.kicad_sch (KiCad schematic)
At the start: 9 parts, among them J1 POGO_Conn, SW1 TL1105SF160Q, SW2 TL1105SF160Q, U2 NanoS3

Commit message: Added Charging Sense Circuit
Added charging sense circuit to allow for detecting if the circuit is turned on using an IO pin on the MCU
Parts:
- added D2: LED, symbol Device:LED
- added Q1: Q_PMOS_GSD, symbol Device:Q_PMOS_GSD
- added R2: 3.3k, symbol Device:R
Connections:
- net +5V: now also R2.1
- net STAT: now reaches U2.1 (STAT)
- net STAT: now also D2.1 (K), Q1.1 (G)
- net IO17: now reaches U2.12 (IO17)
- net IO17: now also Q1.3 (D)
- new net: D2.2 (A), R2.2
- new net +3.3V: Q1.2 (S)
- no-connect marks 17 -> 15
Other:
- moved on the sheet: TFT_SCR2

Commit message: Updated Symbols Footrprints and Routing
Updated the symbols, footprints and the PCB routing to work with the new resistors and ADC circuit
Parts:
- removed C1: JMK105BJ105KV-F, JMK105BJ105KV-F:CAPC1005X55N, symbol Device:JMK105BJ105KV-F
- removed D2: LED, symbol Device:LED
- removed Q1: Q_PMOS_GSD, symbol Device:Q_PMOS_GSD
- removed R1: RC1206FR-0710KL, RC1206FR-0710KL:RESC3116X65N, symbol Device:RC1206FR-0710KL
- added R3: 50k, RT0603BRD0750KL:RESC1608X55N, symbol Device:R
- added R4: 442k, RMCF0402FT442K:RESC1005X35N, symbol Device:R
- added R5: 160k, RC0402FR-07160KL:RESC1005X40N, symbol Device:R
- R2: value 3.3k -> 50k; footprint (none) -> RT0603BRD0750KL:RESC1608X55N
Connections:
- net GND: now also R3.2, R5.2
- net IO17: now also R2.2, R3.1; no longer U2.12 (IO17)
- net VBAT: now also R4.1
- net IO1: now reaches U2.33 (IO1)
- net IO1: now also R4.2, R5.1
Other:
- moved on the sheet: R2

Commit message: Changed The FPC Connector To A Smaller Pitch
Changed the FPC connector on the PCB so that the pitch is reduced and overall footprint is minimized as much as possible
Parts:
- J1: footprint Connector_FFC-FPC:TE_84952-4_1x04-1MP_P1.0mm_Horizontal -> Connector:AMPHENOL_59453-042110ECHLF
Changed lines of the file:
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@@
       (effects (font (size 1.27 1.27)))
     )
-    (property "Footprint" "Connector_FFC-FPC:TE_84952-4_1x04-1MP_P1.0mm_Horizontal" (at 195.58 99.06 0)
+    (property "Footprint" "Connector:AMPHENOL_59453-042110ECHLF" (at 195.58 99.06 0)
       (effects (font (size 1.27 1.27)) hide)
     )

Commit message: Added New PCB Conenctors, Routes, Components
Added new PCB components to reduce the height, changed the traces and adjusted for the battery in the PCB
Parts:
- removed BT2: Battery, Connector_JST:JST_ACH_BM02B-ACHSS-GAN-ETF_1x02-1MP_P1.20mm_Vertical, symbol Device:Battery
- removed J1: POGO_Conn, Connector:AMPHENOL_59453-042110ECHLF, symbol Connector:Conn_01x04_Socket
- removed SW1, SW2: TL1105SF160Q, TL1105SF160Q:SW_TL1105SF160Q, symbol Switch:TL1105SF160Q
- added BT1: Battery, Connector_JST:JST_ACH_BM02B-ACHSS-GAN-ETF_1x02-1MP_P1.20mm_Vertical, symbol Device:Battery
- added D+1, D-1, GND1, PWR1: TestPoint, TestPoint:TestPoint_Pad_D1.0mm, symbol Connector:TestPoint
- added S1, S2: TL1014BF160QG, TL1014BF160QG:TL1014BF160QG, symbol Device:TL1014BF160QG
Connections:
- net D+: now also D+1.1
- net D-: now also D-1.1
- net GND: now also BT1.2 (-), GND1.1, S1.1, S1.3, S2.2, S2.4
- net IO0: now also S2.1, S2.3
- net IO17: now also U2.12 (IO17)
- net RESET: now also S1.2, S1.4
- net VBAT: now also BT1.1 (+)
- net at D1.2 (A): now also PWR1.1
- no-connect marks 15 -> 14
Other:
- note removed: "D+"
- note removed: "D-"
